File: pcb/klaptik-fx.kicad_sch (KiCad schematic)
At the start: 30 parts, among them J1 QWIIC, J2 TagConnect, J3 Conn_01x06, J4 Conn_01x06, J5 IO_B, J6 IO_A, U1 STM32G0xxFx, U2 LCD12864, U3 M95M01-DF

Commit message: rev 0x03
Parts:
- removed C7, C8: 100nF, Resistor_SMD:R_0603_1608Metric, symbol Device:C
- removed J2: TagConnect, Connector:Tag-Connect_TC2030-IDC-NL_2x03_P1.27mm_Vertical, symbol @jb:TagConnect
- removed J3, J4: Conn_01x06, Footprints:SolderConnector, symbol Connector_Generic:Conn_01x06
- removed J5: IO_B, Connector_JST:JST_SH_SM05B-SRSS-TB_1x05-1MP_P1.00mm_Horizontal, symbol Connector_Generic:Conn_01x05
- removed J6: IO_A, Connector_JST:JST_SH_SM04B-SRSS-TB_1x04-1MP_P1.00mm_Horizontal, symbol Connector_Generic:Conn_01x04
- removed R11: DNP, Resistor_SMD:R_0603_1608Metric, symbol Device:R
- removed RN1, RN2: 190Ω, Resistor_SMD:R_Array_Convex_4x0603, symbol Device:R_Pack04
- removed U1: STM32G0xxFx, Package_SO:TSSOP-20_4.4x6.5mm_P0.65mm, symbol @jb:STM32G0xxFx
- added F1: Polyfuse, Fuse:Fuse_0402_1005Metric, symbol Device:Polyfuse
- added J1: 5V, Connector_PinHeader_2.54mm:PinHeader_1x02_P2.54mm_Vertical, symbol Connector_Generic:Conn_01x02
- added J2: BAT, Connector_JST:JST_SH_SM03B-SRSS-TB_1x03-1MP_P1.00mm_Horizontal, symbol Connector_Generic:Conn_01x03
- added J3: FFC, Connector_FFC-FPC:Molex_54548-1071_1x10-1MP_P0.5mm_Horizontal, symbol Connector_Generic:Conn_01x10
- added J4: Header, Connector_PinHeader_1.27mm:PinHeader_1x10_P1.27mm_Vertical, symbol Connector_Generic:Conn_01x10
- added R1: 10KΩ, Resistor_SMD:R_0402_1005Metric, symbol Device:R
- added R2, R9: DNP, Resistor_SMD:R_0402_1005Metric, symbol Device:R
- added TP1: VDD, TestPoint:TestPoint_Pad_D1.0mm, symbol Connector:TestPoint
- added TP2, TP3: GND, TestPoint:TestPoint_Pad_D1.0mm, symbol Connector:TestPoint
- added TP4: SWD IO, TestPoint:TestPoint_Pad_D1.0mm, symbol Connector:TestPoint
- added TP5: SWD CLK, TestPoint:TestPoint_Pad_D1.0mm, symbol Connector:TestPoint
- added U1: AP7370-33W5-7, Package_TO_SOT_SMD:TSOT-23-5, symbol @jb:AP7370-33W5-7
- added U2: AP22652_3x, Package_TO_SOT_SMD:SOT-23-6, symbol @jb:AP22652_3x
- added U3: MP2667GG, @jb:MP2667GG-xxxx-Z, symbol @jb:MP2667GG-xxxx-Z
- added U5: STM32G041G8Ux, Package_DFN_QFN:QFN-28_4x4mm_P0.5mm, symbol MCU_ST_STM32G0:STM32G041G8Ux
- C1: value 10uF -> 4.7uF; footprint Resistor_SMD:R_0603_1608Metric -> Capacitor_SMD:C_0402_1005Metric
- C2, C3, C4, C6: value 100nF -> 4.7uF; footprint Resistor_SMD:R_0603_1608Metric -> Capacitor_SMD:C_0402_1005Metric
- C5: footprint Resistor_SMD:R_0603_1608Metric -> Capacitor_SMD:C_0402_1005Metric
- R10: renamed from R1; value 4.7KΩ -> 2.2KΩ; footprint Resistor_SMD:R_0603_1608Metric -> Resistor_SMD:R_0402_1005Metric
- R11: renamed from R2; value 4.7KΩ -> 2.2KΩ; footprint Resistor_SMD:R_0603_1608Metric -> Resistor_SMD:R_0402_1005Metric
- R12: renamed from R9; footprint Resistor_SMD:R_0603_1608Metric -> Resistor_SMD:R_0402_1005Metric
- R13: renamed from R10; footprint Resistor_SMD:R_0603_1608Metric -> Resistor_SMD:R_0402_1005Metric
- R3: value 10KΩ -> 100KΩ; footprint Resistor_SMD:R_0603_1608Metric -> Resistor_SMD:R_0402_1005Metric
- R4, R6: value 10KΩ -> 20KΩ; footprint Resistor_SMD:R_0603_1608Metric -> Resistor_SMD:R_0402_1005Metric
- R5, R7: footprint Resistor_SMD:R_0603_1608Metric -> Resistor_SMD:R_0402_1005Metric
- R8: value 10KΩ -> 0Ω; footprint Resistor_SMD:R_0603_1608Metric -> Resistor_SMD:R_0402_1005Metric
- U6: renamed from U3; value M95M01-DF -> M95512; footprint Package_SO:SO-8_3.9x4.9mm_P1.27mm -> Package_SO:TSSOP-8_4.4x3mm_P0.65mm
- renumbered J1 to J5, U2 to U4
Connections:
- net GPIO_A1 is gone; now on net VDD: C5.1, R5.2
- net GPIO_B2 is gone; now on net GND: R7.2
- net GPIO_B3 is gone; now on net Vdrive: R8.2
- net GND: now also R12.2, R6.2, J1.1 (Pin_1), J2.3 (Pin_3), J3.1 (Pin_1), J4.1 (Pin_1), TP2.1, U1.2 (GND), U2.2 (GND), U3.5 (GND), U5.4 (VSS); no longer U4.13 (LED_K)
- net I2C_SCL: now also R11.2, U3.6 (SCL), U5.18 (PA11/PA9); no longer R10.2
- net I2C_SDA: now also R10.2, U3.7 (SDA), U5.19 (PA12/PA10); no longer R11.2
- net SPI_CLK: now also U5.28 (PB8)
- net SPI_MISO: now also U5.26 (PB6)
- net SPI_MOSI: now also U5.27 (PB7)
- net SWD_CLK: now also TP5.1, U5.21 (PA14)
- net SWD_IO: now also TP4.1, U5.20 (PA13)
- net VDD: now also C3.1, C4.1, R9.2, TP1.1, U1.5 (VOUT), U2.1 (VIN), U5.3 (VDD); no longer C1.1, C2.1, J5.2 (Pin_2), R13.1, R4.1, R5.1, R6.1, R7.1, R8.1, U4.6 (VDD), U6.7 (~{HOLD}), U6.8 (VCC)
- net LCD_BL: now reaches U4.14 (LED_A)
- net LCD_BL: now also U5.15 (PB1); no longer R12.2
- net ~{FLASH_WP}: now reaches R13.2, U6.3 (~{W})
- net ~{FLASH_WP}: now also U5.2 (PC15)
- net FLASH_CS renamed ~{FLASH_CS}
- net ~{FLASH_CS}: now also U5.23 (PB3)
- net GPIO_A2 renamed VCC_SENSE
- net VCC_SENSE: now also R7.1, U5.14 (PB0); no longer C4.1
- net GPIO_B1 renamed Vdrive
- net Vdrive: now also R13.1, U4.6 (VDD), U6.7 (~{HOLD}), U6.8 (VCC), J3.10 (Pin_10), J4.10 (Pin_10), U2.6 (VOUT); no longer R6.2
- net LCD_A0 renamed LCD_DC
- net LCD_DC: now also U5.17 (PC6)
- net LCD_BLK: no longer names the net of R12.1
- net LCD_BLK: now also U4.13 (LED_K)
- net LCD_CS renamed ~{LCD_CS}
- net ~{LCD_CS}: now also U5.22 (PA15)
- net LCD_RESET renamed ~{LCD_RST}
- net ~{LCD_RST}: now also U5.16 (PA8)
- net RESET renamed ~{PWR_INT}
- net ~{PWR_INT}: now also U3.3 (INT), U5.25 (PB5); no longer C3.1
- new net: J5.2 (Pin_2), R8.1, R9.1
- new net: R6.1, U2.5 (ILIM)
- new net: J2.2 (Pin_2), R1.2, U3.2 (NTC)
- new net: C2.1, U3.4 (VDD)
- new net: F1.1, J1.2 (Pin_2)
- new net BAT+: J2.1 (Pin_1), U3.8 (BATT), U3.9 (BATT)
- new net IO0: J3.2 (Pin_2), J4.2 (Pin_2), U5.6 (PA0)
- new net IO1: J3.3 (Pin_3), J4.3 (Pin_3), U5.7 (PA1)
- new net IO2: J3.4 (Pin_4), J4.4 (Pin_4), U5.8 (PA2)
- new net IO3: J3.5 (Pin_5), J4.5 (Pin_5), U5.9 (PA3)
- new net IO4: J3.6 (Pin_6), J4.6 (Pin_6), U5.10 (PA4)
- new net IO5: J3.7 (Pin_7), J4.7 (Pin_7), U5.11 (PA5)
- new net IO6: J3.8 (Pin_8), J4.8 (Pin_8), U5.12 (PA6)
- new net IO7: J3.9 (Pin_9), J4.9 (Pin_9), U5.13 (PA7)
- new net PRW_EN: U2.3 (EN), U5.24 (PB4)
- new net VCC: C1.1, R2.1, R4.1, U1.1 (VIN), U3.10 (SYS)
- new net V_{in}: F1.2, R1.1, R2.2, U3.1 (IN)
- new net ~{PWR_FLT}: R5.1, U2.4 (FAULT), U5.1 (PC14)
- new net ~{RST}: TP3.1, U5.5 (PF2)
- no-connect marks 2 -> 0
Other:
- moved on the sheet: J5, R10, R11, R12, R13, U4, U6

Commit message: update schematics
Parts:
- R6: value 20KΩ -> 200KΩ
Changed lines of the file:
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@@
       (effects (font (size 1.27 1.27)) (justify left))
     )
-    (property "Value" "20KΩ" (at 257.81 59.69 0)
+    (property "Value" "200KΩ" (at 257.81 59.69 0)
       (effects (font (size 1.27 1.27)) (justify left))
     )
